File: _autosave-placa sensor de mangal.sch (KiCad schematic (older format))
At the start: 4 parts, among them J1 3, J2 1, J3 2

Commit message: upgrade
Parts:
- J1, J2, J3: footprint Connector_Pin:Pin_D1.0mm_L10.0mm -> Connector_Pin:Pin_D1.4mm_L8.5mm_W2.8mm_FlatFork
Changed lines of the file:
@@
 F 0 "J2" H 2688 2036 50  0000 C CNN
 F 1 "1" H 2688 1945 50  0000 C CNN
-F 2 "Connector_Pin:Pin_D1.0mm_L10.0mm" H 2580 1855 50  0001 C CNN
+F 2 "Connector_Pin:Pin_D1.4mm_L8.5mm_W2.8mm_FlatFork" H 2580 1855 50  0001 C CNN
 F 3 "~" H 2580 1855 50  0001 C CNN
 	1    2580 1855
@@
 F 0 "J3" H 2698 2366 50  0000 C CNN
 F 1 "2" H 2698 2275 50  0000 C CNN
-F 2 "Connector_Pin:Pin_D1.0mm_L10.0mm" H 2590 2185 50  0001 C CNN
+F 2 "Connector_Pin:Pin_D1.4mm_L8.5mm_W2.8mm_FlatFork" H 2590 2185 50  0001 C CNN
 F 3 "~" H 2590 2185 50  0001 C CNN
 	1    2590 2185
@@
 F 0 "J1" H 2678 2741 50  0000 C CNN
 F 1 "3" H 2678 2650 50  0000 C CNN
-F 2 "Connector_Pin:Pin_D1.0mm_L10.0mm" H 2570 2560 50  0001 C CNN
+F 2 "Connector_Pin:Pin_D1.4mm_L8.5mm_W2.8mm_FlatFork" H 2570 2560 50  0001 C CNN
 F 3 "~" H 2570 2560 50  0001 C CNN
 	1    2570 2560
