File: placa sensor de mangal.sch (KiCad schematic (older format))
At the start: 4 parts

Commit message: upgrade
Parts:
- removed J?: 2, Connector:Banana_Jack_1Pin, symbol Connector:Conn_01x01_Male
- removed J?: 3, Connector:Banana_Jack_1Pin, symbol Connector:Conn_01x01_Male
- added J1: 3, Connector_Pin:Pin_D1.4mm_L8.5mm_W2.8mm_FlatFork, symbol Connector:Conn_01x01_Male
- added J3: 2, Connector_Pin:Pin_D1.4mm_L8.5mm_W2.8mm_FlatFork, symbol Connector:Conn_01x01_Male
- J2: renamed from J?; footprint Connector:Banana_Jack_1Pin -> Connector_Pin:Pin_D1.4mm_L8.5mm_W2.8mm_FlatFork
- TH1: renamed from TH?; footprint Resistor_THT:R_Axial_DIN0204_L3.6mm_D1.6mm_P2.54mm_Vertical -> Resistor_THT:R_Axial_DIN0204_L3.6mm_D1.6mm_P5.08mm_Horizontal
Connections:
- net at J2.1 (Pin_1), TH1.1: now also J3.1 (Pin_1)
- net at TH1.2: now also J1.1 (Pin_1)
Changed lines of the file:
@@
 $EndDescr
 $Comp
-L Connector:Conn_01x01_Male J?
+L Connector:Conn_01x01_Male J2
 U 1 1 608C9C7F
 P 2580 1855
-F 0 "J?" H 2688 2036 50  0000 C CNN
+F 0 "J2" H 2688 2036 50  0000 C CNN
 F 1 "1" H 2688 1945 50  0000 C CNN
-F 2 "Connector:Banana_Jack_1Pin" H 2580 1855 50  0001 C CNN
+F 2 "Connector_Pin:Pin_D1.4mm_L8.5mm_W2.8mm_FlatFork" H 2580 1855 50  0001 C CNN
 F 3 "~" H 2580 1855 50  0001 C CNN
 	1    2580 1855
@@
 $EndComp
 $Comp
-L Connector:Conn_01x01_Male J?
-U 1 1 608CA207
-P 2590 2185
-F 0 "J?" H 2698 2366 50  0000 C CNN
-F 1 "2" H 2698 2275 50  0000 C CNN
-F 2 "Connector:Banana_Jack_1Pin" H 2590 2185 50  0001 C CNN
-F 3 "~" H 2590 2185 50  0001 C CNN
-	1    2590 2185
-	1    0    0    -1
-$EndComp
-$Comp
-L Connector:Conn_01x01_Male J?
-U 1 1 608CA89A
-P 2570 2560
-F 0 "J?" H 2678 2741 50  0000 C CNN
-F 1 "3" H 2678 2650 50  0000 C CNN
-F 2 "Connector:Banana_Jack_1Pin" H 2570 2560 50  0001 C CNN
-F 3 "~" H 2570 2560 50  0001 C CNN
-	1    2570 2560
-	1    0    0    -1
-$EndComp
-$Comp
-L Sensor_Temperature:PT100 TH?
+L Sensor_Temperature:PT100 TH1
 U 1 1 608CAFBE
 P 3475 2365
-F 0 "TH?" H 3573 2411 50  0000 L CNN
+F 0 "TH1" H 3573 2411 50  0000 L CNN
 F 1 "PT100" H 3573 2320 50  0000 L CNN
-F 2 "Resistor_THT:R_Axial_DIN0204_L3.6mm_D1.6mm_P2.54mm_Vertical" H 3475 2415 50  0001 C CNN
+F 2 "Resistor_THT:R_Axial_DIN0204_L3.6mm_D1.6mm_P5.08mm_Horizontal" H 3475 2415 50  0001 C CNN
 F 3 "https://www.heraeus.com/media/media/group/doc_group/products_1/hst/sot_to/de_15/to_92_d.pdf" H 3475 2415 50  0001 C CNN
 	1    3475 2365
@@
 Wire Wire Line
 	3160 1855 2780 1855
+$Comp
+L Connector:Conn_01x01_Male J3
+U 1 1 608CD9CF
+P 2590 2185
+F 0 "J3" H 2698 2366 50  0000 C CNN
+F 1 "2" H 2698 2275 50  0000 C CNN
+F 2 "Connector_Pin:Pin_D1.4mm_L8.5mm_W2.8mm_FlatFork" H 2590 2185 50  0001 C CNN
+F 3 "~" H 2590 2185 50  0001 C CNN
+	1    2590 2185
+	1    0    0    -1
+$EndComp
+$Comp
+L Connector:Conn_01x01_Male J1
+U 1 1 608CE0CB
+P 2570 2560
+F 0 "J1" H 2678 2741 50  0000 C CNN
+F 1 "3" H 2678 2650 50  0000 C CNN
+F 2 "Connector_Pin:Pin_D1.4mm_L8.5mm_W2.8mm_FlatFork" H 2570 2560 50  0001 C CNN
+F 3 "~" H 2570 2560 50  0001 C CNN
+	1    2570 2560
+	1    0    0    -1
+$EndComp
 $EndSCHEMATC

Commit message: sin cambios
Parts:
- TH1: footprint Resistor_THT:R_Axial_DIN0204_L3.6mm_D1.6mm_P5.08mm_Horizontal -> Resistor_THT:R_Axial_DIN0204_L3.6mm_D1.6mm_P2.54mm_Vertical
Changed lines of the file:
@@
 F 0 "TH1" H 3573 2411 50  0000 L CNN
 F 1 "PT100" H 3573 2320 50  0000 L CNN
-F 2 "Resistor_THT:R_Axial_DIN0204_L3.6mm_D1.6mm_P5.08mm_Horizontal" H 3475 2415 50  0001 C CNN
+F 2 "Resistor_THT:R_Axial_DIN0204_L3.6mm_D1.6mm_P2.54mm_Vertical" H 3475 2415 50  0001 C CNN
 F 3 "https://www.heraeus.com/media/media/group/doc_group/products_1/hst/sot_to/de_15/to_92_d.pdf" H 3475 2415 50  0001 C CNN
 	1    3475 2365
