File: placa sensor de mangal.kicad_pcb (KiCad board)
At the start: 2 copper layers, 9.1 x 13.5 mm, 4 parts, among them J1 3, J2 1, J3 2

Commit message: upgrade
Parts:
- J1, J2, J3: footprint Connector_Pin:Pin_D1.0mm_L10.0mm -> Connector_Pin:Pin_D1.4mm_L8.5mm_W2.8mm_FlatFork
- moved TH1 0.52 mm to (141.6, 105.3)
- moved J2 0.46 mm to (140.3, 95.8)
- moved J3 0.18 mm to (140.2, 100.6)
- moved J1 0.13 mm to (145.2, 98.2)
Routing:
- net Net-(J2-Pad1): track 9.21 -> 10.2 mm
- net Net-(J1-Pad1): track 6.95 -> 7.53 mm

Commit message: sin cambios
Parts:
- moved J1 0.89 mm to (146.1, 98.2)
- moved J3 0.89 mm to (141.1, 100.6)
- moved TH1 0.89 mm to (142.5, 105.3)
- moved J2 0.89 mm to (141.2, 95.8)
